File: project/batfind/filt_in_audio.sch (KiCad schematic (older format))
At the start: 0 parts

Commit message: Schematic updated
Parts:
- added C?: 1n, symbol C
- added C?: 4.7u, symbol C
- added R?: 1k, symbol R
- added R?: 10k, symbol R
- added U?: OPA835, symbol OPA835
Connections:
- net filt_in: now also R?.2
- net filt_out: now also C?.1, R?.1
- new net: C?.1, R?.1, U?.3 (IN+)
- new net: C?.2, U?.1 (OUT), U?.4 (IN-)
- new net GND: C?.2, R?.2, U?.2 (VS-)
- new net VCC: U?.5 (PD), U?.6 (VS+)
Changed lines of the file:
@@
 Comment4 ""
 $EndDescr
-Text HLabel 4100 4000 0    60   Input ~ 0
+Text HLabel 4050 4000 0    60   Input ~ 0
 filt_in
-Text HLabel 6750 4000 2    60   Output ~ 0
+Text HLabel 6900 3850 2    60   Output ~ 0
 filt_out
+Text HLabel 4050 4650 0    60   Input ~ 0
+ref
+$Comp
+L R R?
+U 1 1 547B9FF3
+P 4400 4000
+F 0 "R?" V 4480 4000 40  0000 C CNN
+F 1 "1k" V 4407 4001 40  0000 C CNN
+F 2 "" V 4330 4000 30  0000 C CNN
+F 3 "" H 4400 4000 30  0000 C CNN
+	1    4400 4000
+	0    1    1    0
+$EndComp
+$Comp
+L C C?
+U 1 1 547BA03D
+P 4750 4250
+F 0 "C?" H 4750 4350 40  0000 L CNN
+F 1 "1n" H 4756 4165 40  0000 L CNN
+F 2 "" H 4788 4100 30  0000 C CNN
+F 3 "" H 4750 4250 60  0000 C CNN
+	1    4750 4250
+	1    0    0    -1
+$EndComp
+$Comp
+L OPA835 U?
+U 1 1 547BA070
+P 5400 3850
+F 0 "U?" H 5700 4000 60  0000 C CNN
+F 1 "OPA835" H 5800 3700 60  0000 C CNN
+F 2 "" H 5800 3700 60  0000 C CNN
+F 3 "" H 5800 3700 60  0000 C CNN
+	1    5400 3850
+	1    0    0    -1
+$EndComp
+$Comp
+L R R?
+U 1 1 547BA0AE
+P 6700 4200
+F 0 "R?" V 6780 4200 40  0000 C CNN
+F 1 "10k" V 6707 4201 40  0000 C CNN
+F 2 "" V 6630 4200 30  0000 C CNN
+F 3 "" H 6700 4200 30  0000 C CNN
+	1    6700 4200
+	1    0    0    -1
+$EndComp
+$Comp
+L C C?
+U 1 1 547BA0F3
+P 6350 3850
+F 0 "C?" H 6350 3950 40  0000 L CNN
+F 1 "4.7u" H 6356 3765 40  0000 L CNN
+F 2 "" H 6388 3700 30  0000 C CNN
+F 3 "" H 6350 3850 60  0000 C CNN
+	1    6350 3850
+	0    1    1    0
+$EndComp
+Wire Wire Line
+	4050 4000 4150 4000
+Wire Wire Line
+	4650 4000 4900 4000
+Wire Wire Line
+	4750 4050 4750 4000
+Connection ~ 4750 4000
+Wire Wire Line
+	4900 3700 4800 3700
+Wire Wire Line
+	4800 3700 4800 3250
+Wire Wire Line
+	4800 3250 6050 3250
+Wire Wire Line
+	6050 3250 6050 3850
+Wire Wire Line
+	6000 3850 6150 3850
+Connection ~ 6050 3850
+Wire Wire Line
+	6550 3850 6900 3850
+Wire Wire Line
+	6700 3850 6700 3950
+Connection ~ 6700 3850
+$Comp
+L GND #PWR?
+U 1 1 547BA732
+P 5350 4250
+F 0 "#PWR?" H 5350 4250 30  0001 C CNN
+F 1 "GND" H 5350 4180 30  0001 C CNN
+F 2 "" H 5350 4250 60  0000 C CNN
+F 3 "" H 5350 4250 60  0000 C CNN
+	1    5350 4250
+	1    0    0    -1
+$EndComp
+$Comp
+L GND #PWR?
+U 1 1 547BA74B
+P 4750 4450
+F 0 "#PWR?" H 4750 4450 30  0001 C CNN
+F 1 "GND" H 4750 4380 30  0001 C CNN
+F 2 "" H 4750 4450 60  0000 C CNN
+F 3 "" H 4750 4450 60  0000 C CNN
+	1    4750 4450
+	1    0    0    -1
+$EndComp
+$Comp
+L GND #PWR?
+U 1 1 547BA764
+P 6700 4450
+F 0 "#PWR?" H 6700 4450 30  0001 C CNN
+F 1 "GND" H 6700 4380 30  0001 C CNN
+F 2 "" H 6700 4450 60  0000 C CNN
+F 3 "" H 6700 4450 60  0000 C CNN
+	1    6700 4450
+	1    0    0    -1
+$EndComp
+$Comp
+L VCC #PWR?
+U 1 1 547BA77D
+P 5350 3450
+F 0 "#PWR?" H 5350 3550 30  0001 C CNN
+F 1 "VCC" H 5350 3550 30  0000 C CNN
+F 2 "" H 5350 3450 60  0000 C CNN
+F 3 "" H 5350 3450 60  0000 C CNN
+	1    5350 3450
+	1    0    0    -1
+$EndComp
+$Comp
+L VCC #PWR?
+U 1 1 547BA7AF
+P 5550 4150
+F 0 "#PWR?" H 5550 4250 30  0001 C CNN
+F 1 "VCC" H 5550 4250 30  0000 C CNN
+F 2 "" H 5550 4150 60  0000 C CNN
+F 3 "" H 5550 4150 60  0000 C CNN
+	1    5550 4150
+	-1   0    0    1
+$EndComp
 $EndSCHEMATC

Commit message: Schematic annotated and netlist generated
Parts:
- gave numbers to parts that had none: 5
Changed lines of the file:
@@
 ref
 $Comp
-L R R?
+L R R19
 U 1 1 547B9FF3
 P 4400 4000
-F 0 "R?" V 4480 4000 40  0000 C CNN
+F 0 "R19" V 4480 4000 40  0000 C CNN
 F 1 "1k" V 4407 4001 40  0000 C CNN
 F 2 "" V 4330 4000 30  0000 C CNN
@@
 $EndComp
 $Comp
-L C C?
+L C C17
 U 1 1 547BA03D
 P 4750 4250
-F 0 "C?" H 4750 4350 40  0000 L CNN
+F 0 "C17" H 4750 4350 40  0000 L CNN
 F 1 "1n" H 4756 4165 40  0000 L CNN
 F 2 "" H 4788 4100 30  0000 C CNN
@@
 $EndComp
 $Comp
-L OPA835 U?
+L OPA835 U9
 U 1 1 547BA070
 P 5400 3850
-F 0 "U?" H 5700 4000 60  0000 C CNN
+F 0 "U9" H 5700 4000 60  0000 C CNN
 F 1 "OPA835" H 5800 3700 60  0000 C CNN
 F 2 "" H 5800 3700 60  0000 C CNN
@@
 $EndComp
 $Comp
-L R R?
+L R R20
 U 1 1 547BA0AE
 P 6700 4200
-F 0 "R?" V 6780 4200 40  0000 C CNN
+F 0 "R20" V 6780 4200 40  0000 C CNN
 F 1 "10k" V 6707 4201 40  0000 C CNN
 F 2 "" V 6630 4200 30  0000 C CNN
@@
 $EndComp
 $Comp
-L C C?
+L C C18
 U 1 1 547BA0F3
 P 6350 3850
-F 0 "C?" H 6350 3950 40  0000 L CNN
+F 0 "C18" H 6350 3950 40  0000 L CNN
 F 1 "4.7u" H 6356 3765 40  0000 L CNN
 F 2 "" H 6388 3700 30  0000 C CNN
@@
 Connection ~ 6700 3850
 $Comp
-L GND #PWR?
+L GND #PWR042
 U 1 1 547BA732
 P 5350 4250
-F 0 "#PWR?" H 5350 4250 30  0001 C CNN
+F 0 "#PWR042" H 5350 4250 30  0001 C CNN
 F 1 "GND" H 5350 4180 30  0001 C CNN
 F 2 "" H 5350 4250 60  0000 C CNN
@@
 $EndComp
 $Comp
-L GND #PWR?
+L GND #PWR043
 U 1 1 547BA74B
 P 4750 4450
-F 0 "#PWR?" H 4750 4450 30  0001 C CNN
+F 0 "#PWR043" H 4750 4450 30  0001 C CNN
 F 1 "GND" H 4750 4380 30  0001 C CNN
 F 2 "" H 4750 4450 60  0000 C CNN
@@
 $EndComp
 $Comp
-L GND #PWR?
+L GND #PWR044
 U 1 1 547BA764
 P 6700 4450
-F 0 "#PWR?" H 6700 4450 30  0001 C CNN
+F 0 "#PWR044" H 6700 4450 30  0001 C CNN
 F 1 "GND" H 6700 4380 30  0001 C CNN
 F 2 "" H 6700 4450 60  0000 C CNN
@@
 $EndComp
 $Comp
-L VCC #PWR?
+L VCC #PWR045
 U 1 1 547BA77D
 P 5350 3450
-F 0 "#PWR?" H 5350 3550 30  0001 C CNN
+F 0 "#PWR045" H 5350 3550 30  0001 C CNN
 F 1 "VCC" H 5350 3550 30  0000 C CNN
 F 2 "" H 5350 3450 60  0000 C CNN
@@
 $EndComp
 $Comp
-L VCC #PWR?
+L VCC #PWR046
 U 1 1 547BA7AF
 P 5550 4150
-F 0 "#PWR?" H 5550 4250 30  0001 C CNN
+F 0 "#PWR046" H 5550 4250 30  0001 C CNN
 F 1 "VCC" H 5550 4250 30  0000 C CNN
 F 2 "" H 5550 4150 60  0000 C CNN
