File: project/batfind/filt_in_us.sch (KiCad schematic (older format))
At the start: 0 parts

Commit message: Schematic updated
Parts:
- added C?: 1n, symbol C
- added C?: 22n, symbol C
- added R?: 470, symbol R
- added R?: 1k, symbol R
- added U?: OPA835, symbol OPA835
Connections:
- net filt_in: now also R?.2
- net filt_out: now also C?.1, R?.1
- new net: C?.1, R?.1, U?.3 (IN+)
- new net: C?.2, U?.1 (OUT), U?.4 (IN-)
- new net GND: C?.2, R?.2, U?.2 (VS-)
- new net VCC: U?.5 (PD), U?.6 (VS+)
Changed lines of the file:
@@
 Comment4 ""
 $EndDescr
-Text HLabel 4800 3800 0    60   Input ~ 0
+Text HLabel 4550 3800 0    60   Input ~ 0
 filt_in
-Text HLabel 7450 3800 2    60   Output ~ 0
+Text HLabel 7150 3650 2    60   Output ~ 0
 filt_out
+Text HLabel 4800 4150 0    60   Input ~ 0
+ref
+$Comp
+L C C?
+U 1 1 547BA893
+P 5250 4100
+F 0 "C?" H 5250 4200 40  0000 L CNN
+F 1 "1n" H 5256 4015 40  0000 L CNN
+F 2 "" H 5288 3950 30  0000 C CNN
+F 3 "" H 5250 4100 60  0000 C CNN
+	1    5250 4100
+	1    0    0    -1
+$EndComp
+$Comp
+L C C?
+U 1 1 547BA8D5
+P 6700 3650
+F 0 "C?" H 6700 3750 40  0000 L CNN
+F 1 "22n" H 6706 3565 40  0000 L CNN
+F 2 "" H 6738 3500 30  0000 C CNN
+F 3 "" H 6700 3650 60  0000 C CNN
+	1    6700 3650
+	0    1    1    0
+$EndComp
+$Comp
+L OPA835 U?
+U 1 1 547BA926
+P 5800 3650
+F 0 "U?" H 6100 3800 60  0000 C CNN
+F 1 "OPA835" H 6200 3500 60  0000 C CNN
+F 2 "" H 6200 3500 60  0000 C CNN
+F 3 "" H 6200 3500 60  0000 C CNN
+	1    5800 3650
+	1    0    0    -1
+$EndComp
+$Comp
+L R R?
+U 1 1 547BA988
+P 4950 3800
+F 0 "R?" V 5030 3800 40  0000 C CNN
+F 1 "470" V 4957 3801 40  0000 C CNN
+F 2 "" V 4880 3800 30  0000 C CNN
+F 3 "" H 4950 3800 30  0000 C CNN
+	1    4950 3800
+	0    1    1    0
+$EndComp
+$Comp
+L R R?
+U 1 1 547BAA5E
+P 7000 3950
+F 0 "R?" V 7080 3950 40  0000 C CNN
+F 1 "1k" V 7007 3951 40  0000 C CNN
+F 2 "" V 6930 3950 30  0000 C CNN
+F 3 "" H 7000 3950 30  0000 C CNN
+	1    7000 3950
+	1    0    0    -1
+$EndComp
+Wire Wire Line
+	4550 3800 4700 3800
+Wire Wire Line
+	5200 3800 5300 3800
+Wire Wire Line
+	5250 3800 5250 3900
+Connection ~ 5250 3800
+Wire Wire Line
+	5200 3500 5300 3500
+Wire Wire Line
+	5200 3000 5200 3500
+Wire Wire Line
+	5200 3000 6450 3000
+Wire Wire Line
+	6450 3000 6450 3650
+Wire Wire Line
+	6400 3650 6500 3650
+Connection ~ 6450 3650
+Wire Wire Line
+	6900 3650 7150 3650
+Wire Wire Line
+	7000 3650 7000 3700
+Connection ~ 7000 3650
+$Comp
+L GND #PWR?
+U 1 1 547BAB1B
+P 7000 4200
+F 0 "#PWR?" H 7000 4200 30  0001 C CNN
+F 1 "GND" H 7000 4130 30  0001 C CNN
+F 2 "" H 7000 4200 60  0000 C CNN
+F 3 "" H 7000 4200 60  0000 C CNN
+	1    7000 4200
+	1    0    0    -1
+$EndComp
+$Comp
+L GND #PWR?
+U 1 1 547BAB34
+P 5250 4300
+F 0 "#PWR?" H 5250 4300 30  0001 C CNN
+F 1 "GND" H 5250 4230 30  0001 C CNN
+F 2 "" H 5250 4300 60  0000 C CNN
+F 3 "" H 5250 4300 60  0000 C CNN
+	1    5250 4300
+	1    0    0    -1
+$EndComp
+$Comp
+L GND #PWR?
+U 1 1 547BAB5C
+P 5750 4050
+F 0 "#PWR?" H 5750 4050 30  0001 C CNN
+F 1 "GND" H 5750 3980 30  0001 C CNN
+F 2 "" H 5750 4050 60  0000 C CNN
+F 3 "" H 5750 4050 60  0000 C CNN
+	1    5750 4050
+	1    0    0    -1
+$EndComp
+$Comp
+L VCC #PWR?
+U 1 1 547BAB75
+P 5750 3250
+F 0 "#PWR?" H 5750 3350 30  0001 C CNN
+F 1 "VCC" H 5750 3350 30  0000 C CNN
+F 2 "" H 5750 3250 60  0000 C CNN
+F 3 "" H 5750 3250 60  0000 C CNN
+	1    5750 3250
+	1    0    0    -1
+$EndComp
+$Comp
+L VCC #PWR?
+U 1 1 547BAB8E
+P 5950 3950
+F 0 "#PWR?" H 5950 4050 30  0001 C CNN
+F 1 "VCC" H 5950 4050 30  0000 C CNN
+F 2 "" H 5950 3950 60  0000 C CNN
+F 3 "" H 5950 3950 60  0000 C CNN
+	1    5950 3950
+	-1   0    0    1
+$EndComp
 $EndSCHEMATC

Commit message: Schematic annotated and netlist generated
Parts:
- gave numbers to parts that had none: 5
Changed lines of the file:
@@
 ref
 $Comp
-L C C?
+L C C15
 U 1 1 547BA893
 P 5250 4100
-F 0 "C?" H 5250 4200 40  0000 L CNN
+F 0 "C15" H 5250 4200 40  0000 L CNN
 F 1 "1n" H 5256 4015 40  0000 L CNN
 F 2 "" H 5288 3950 30  0000 C CNN
@@
 $EndComp
 $Comp
-L C C?
+L C C16
 U 1 1 547BA8D5
 P 6700 3650
-F 0 "C?" H 6700 3750 40  0000 L CNN
+F 0 "C16" H 6700 3750 40  0000 L CNN
 F 1 "22n" H 6706 3565 40  0000 L CNN
 F 2 "" H 6738 3500 30  0000 C CNN
@@
 $EndComp
 $Comp
-L OPA835 U?
+L OPA835 U8
 U 1 1 547BA926
 P 5800 3650
-F 0 "U?" H 6100 3800 60  0000 C CNN
+F 0 "U8" H 6100 3800 60  0000 C CNN
 F 1 "OPA835" H 6200 3500 60  0000 C CNN
 F 2 "" H 6200 3500 60  0000 C CNN
@@
 $EndComp
 $Comp
-L R R?
+L R R17
 U 1 1 547BA988
 P 4950 3800
-F 0 "R?" V 5030 3800 40  0000 C CNN
+F 0 "R17" V 5030 3800 40  0000 C CNN
 F 1 "470" V 4957 3801 40  0000 C CNN
 F 2 "" V 4880 3800 30  0000 C CNN
@@
 $EndComp
 $Comp
-L R R?
+L R R18
 U 1 1 547BAA5E
 P 7000 3950
-F 0 "R?" V 7080 3950 40  0000 C CNN
+F 0 "R18" V 7080 3950 40  0000 C CNN
 F 1 "1k" V 7007 3951 40  0000 C CNN
 F 2 "" V 6930 3950 30  0000 C CNN
@@
 Connection ~ 7000 3650
 $Comp
-L GND #PWR?
+L GND #PWR037
 U 1 1 547BAB1B
 P 7000 4200
-F 0 "#PWR?" H 7000 4200 30  0001 C CNN
+F 0 "#PWR037" H 7000 4200 30  0001 C CNN
 F 1 "GND" H 7000 4130 30  0001 C CNN
 F 2 "" H 7000 4200 60  0000 C CNN
@@
 $EndComp
 $Comp
-L GND #PWR?
+L GND #PWR038
 U 1 1 547BAB34
 P 5250 4300
-F 0 "#PWR?" H 5250 4300 30  0001 C CNN
+F 0 "#PWR038" H 5250 4300 30  0001 C CNN
 F 1 "GND" H 5250 4230 30  0001 C CNN
 F 2 "" H 5250 4300 60  0000 C CNN
@@
 $EndComp
 $Comp
-L GND #PWR?
+L GND #PWR039
 U 1 1 547BAB5C
 P 5750 4050
-F 0 "#PWR?" H 5750 4050 30  0001 C CNN
+F 0 "#PWR039" H 5750 4050 30  0001 C CNN
 F 1 "GND" H 5750 3980 30  0001 C CNN
 F 2 "" H 5750 4050 60  0000 C CNN
@@
 $EndComp
 $Comp
-L VCC #PWR?
+L VCC #PWR040
 U 1 1 547BAB75
 P 5750 3250
-F 0 "#PWR?" H 5750 3350 30  0001 C CNN
+F 0 "#PWR040" H 5750 3350 30  0001 C CNN
 F 1 "VCC" H 5750 3350 30  0000 C CNN
 F 2 "" H 5750 3250 60  0000 C CNN
@@
 $EndComp
 $Comp
-L VCC #PWR?
+L VCC #PWR041
 U 1 1 547BAB8E
 P 5950 3950
-F 0 "#PWR?" H 5950 4050 30  0001 C CNN
+F 0 "#PWR041" H 5950 4050 30  0001 C CNN
 F 1 "VCC" H 5950 4050 30  0000 C CNN
 F 2 "" H 5950 3950 60  0000 C CNN
