File: project/batfind/filt_out_audio.sch (KiCad schematic (older format))
At the start: 0 parts

Commit message: Schematic updated
Parts:
- added C?: 1n, symbol C
- added C?: 4.7u, symbol C
- added R?: 1k, symbol R
- added R?: 10k, symbol R
- added U?: OPA835, symbol OPA835
Connections:
- net filt_in: now also R?.2
- net filt_out: now also C?.1, R?.1
- new net: C?.2, U?.1 (OUT), U?.4 (IN-)
- new net: C?.1, R?.1, U?.3 (IN+)
- new net GND: C?.2, R?.2, U?.2 (VS-)
- new net VCC: U?.5 (PD), U?.6 (VS+)
Changed lines of the file:
@@
 Comment4 ""
 $EndDescr
-Text HLabel 4550 4000 0    60   Input ~ 0
+Text HLabel 4400 4000 0    60   Input ~ 0
 filt_in
-Text HLabel 6900 4000 2    60   Output ~ 0
+Text HLabel 6950 3850 2    60   Output ~ 0
 filt_out
+Text HLabel 4400 4300 0    60   Input ~ 0
+ref
+$Comp
+L OPA835 U?
+U 1 1 547BB8C5
+P 5650 3850
+F 0 "U?" H 5950 4000 60  0000 C CNN
+F 1 "OPA835" H 6050 3700 60  0000 C CNN
+F 2 "" H 6050 3700 60  0000 C CNN
+F 3 "" H 6050 3700 60  0000 C CNN
+	1    5650 3850
+	1    0    0    -1
+$EndComp
+$Comp
+L R R?
+U 1 1 547BB8F9
+P 4750 4000
+F 0 "R?" V 4830 4000 40  0000 C CNN
+F 1 "1k" V 4757 4001 40  0000 C CNN
+F 2 "" V 4680 4000 30  0000 C CNN
+F 3 "" H 4750 4000 30  0000 C CNN
+	1    4750 4000
+	0    1    1    0
+$EndComp
+$Comp
+L C C?
+U 1 1 547BB94E
+P 5050 4250
+F 0 "C?" H 5050 4350 40  0000 L CNN
+F 1 "1n" H 5056 4165 40  0000 L CNN
+F 2 "" H 5088 4100 30  0000 C CNN
+F 3 "" H 5050 4250 60  0000 C CNN
+	1    5050 4250
+	1    0    0    -1
+$EndComp
+$Comp
+L C C?
+U 1 1 547BB971
+P 6550 3850
+F 0 "C?" H 6550 3950 40  0000 L CNN
+F 1 "4.7u" H 6556 3765 40  0000 L CNN
+F 2 "" H 6588 3700 30  0000 C CNN
+F 3 "" H 6550 3850 60  0000 C CNN
+	1    6550 3850
+	0    1    1    0
+$EndComp
+$Comp
+L R R?
+U 1 1 547BB9B6
+P 6850 4200
+F 0 "R?" V 6930 4200 40  0000 C CNN
+F 1 "10k" V 6857 4201 40  0000 C CNN
+F 2 "" V 6780 4200 30  0000 C CNN
+F 3 "" H 6850 4200 30  0000 C CNN
+	1    6850 4200
+	1    0    0    -1
+$EndComp
+Wire Wire Line
+	4400 4000 4500 4000
+Wire Wire Line
+	5000 4000 5150 4000
+Wire Wire Line
+	5050 4000 5050 4050
+Connection ~ 5050 4000
+Wire Wire Line
+	5150 3700 5000 3700
+Wire Wire Line
+	5000 3700 5000 3100
+Wire Wire Line
+	5000 3100 6300 3100
+Wire Wire Line
+	6300 3100 6300 3850
+Wire Wire Line
+	6250 3850 6350 3850
+Connection ~ 6300 3850
+Wire Wire Line
+	6750 3850 6950 3850
+Wire Wire Line
+	6850 3850 6850 3950
+Connection ~ 6850 3850
+$Comp
+L GND #PWR?
+U 1 1 547BBA54
+P 5600 4250
+F 0 "#PWR?" H 5600 4250 30  0001 C CNN
+F 1 "GND" H 5600 4180 30  0001 C CNN
+F 2 "" H 5600 4250 60  0000 C CNN
+F 3 "" H 5600 4250 60  0000 C CNN
+	1    5600 4250
+	1    0    0    -1
+$EndComp
+$Comp
+L GND #PWR?
+U 1 1 547BBA6D
+P 6850 4450
+F 0 "#PWR?" H 6850 4450 30  0001 C CNN
+F 1 "GND" H 6850 4380 30  0001 C CNN
+F 2 "" H 6850 4450 60  0000 C CNN
+F 3 "" H 6850 4450 60  0000 C CNN
+	1    6850 4450
+	1    0    0    -1
+$EndComp
+$Comp
+L GND #PWR?
+U 1 1 547BBA86
+P 5050 4450
+F 0 "#PWR?" H 5050 4450 30  0001 C CNN
+F 1 "GND" H 5050 4380 30  0001 C CNN
+F 2 "" H 5050 4450 60  0000 C CNN
+F 3 "" H 5050 4450 60  0000 C CNN
+	1    5050 4450
+	1    0    0    -1
+$EndComp
+$Comp
+L VCC #PWR?
+U 1 1 547BBACC
+P 5600 3450
+F 0 "#PWR?" H 5600 3550 30  0001 C CNN
+F 1 "VCC" H 5600 3550 30  0000 C CNN
+F 2 "" H 5600 3450 60  0000 C CNN
+F 3 "" H 5600 3450 60  0000 C CNN
+	1    5600 3450
+	1    0    0    -1
+$EndComp
+$Comp
+L VCC #PWR?
+U 1 1 547BBAE5
+P 5800 4150
+F 0 "#PWR?" H 5800 4250 30  0001 C CNN
+F 1 "VCC" H 5800 4250 30  0000 C CNN
+F 2 "" H 5800 4150 60  0000 C CNN
+F 3 "" H 5800 4150 60  0000 C CNN
+	1    5800 4150
+	-1   0    0    1
+$EndComp
 $EndSCHEMATC

Commit message: Schematic annotated and netlist generated
Parts:
- gave numbers to parts that had none: 5
Changed lines of the file:
@@
 ref
 $Comp
-L OPA835 U?
+L OPA835 U6
 U 1 1 547BB8C5
 P 5650 3850
-F 0 "U?" H 5950 4000 60  0000 C CNN
+F 0 "U6" H 5950 4000 60  0000 C CNN
 F 1 "OPA835" H 6050 3700 60  0000 C CNN
 F 2 "" H 6050 3700 60  0000 C CNN
@@
 $EndComp
 $Comp
-L R R?
+L R R13
 U 1 1 547BB8F9
 P 4750 4000
-F 0 "R?" V 4830 4000 40  0000 C CNN
+F 0 "R13" V 4830 4000 40  0000 C CNN
 F 1 "1k" V 4757 4001 40  0000 C CNN
 F 2 "" V 4680 4000 30  0000 C CNN
@@
 $EndComp
 $Comp
-L C C?
+L C C11
 U 1 1 547BB94E
 P 5050 4250
-F 0 "C?" H 5050 4350 40  0000 L CNN
+F 0 "C11" H 5050 4350 40  0000 L CNN
 F 1 "1n" H 5056 4165 40  0000 L CNN
 F 2 "" H 5088 4100 30  0000 C CNN
@@
 $EndComp
 $Comp
-L C C?
+L C C12
 U 1 1 547BB971
 P 6550 3850
-F 0 "C?" H 6550 3950 40  0000 L CNN
+F 0 "C12" H 6550 3950 40  0000 L CNN
 F 1 "4.7u" H 6556 3765 40  0000 L CNN
 F 2 "" H 6588 3700 30  0000 C CNN
@@
 $EndComp
 $Comp
-L R R?
+L R R14
 U 1 1 547BB9B6
 P 6850 4200
-F 0 "R?" V 6930 4200 40  0000 C CNN
+F 0 "R14" V 6930 4200 40  0000 C CNN
 F 1 "10k" V 6857 4201 40  0000 C CNN
 F 2 "" V 6780 4200 30  0000 C CNN
@@
 Connection ~ 6850 3850
 $Comp
-L GND #PWR?
+L GND #PWR027
 U 1 1 547BBA54
 P 5600 4250
-F 0 "#PWR?" H 5600 4250 30  0001 C CNN
+F 0 "#PWR027" H 5600 4250 30  0001 C CNN
 F 1 "GND" H 5600 4180 30  0001 C CNN
 F 2 "" H 5600 4250 60  0000 C CNN
@@
 $EndComp
 $Comp
-L GND #PWR?
+L GND #PWR028
 U 1 1 547BBA6D
 P 6850 4450
-F 0 "#PWR?" H 6850 4450 30  0001 C CNN
+F 0 "#PWR028" H 6850 4450 30  0001 C CNN
 F 1 "GND" H 6850 4380 30  0001 C CNN
 F 2 "" H 6850 4450 60  0000 C CNN
@@
 $EndComp
 $Comp
-L GND #PWR?
+L GND #PWR029
 U 1 1 547BBA86
 P 5050 4450
-F 0 "#PWR?" H 5050 4450 30  0001 C CNN
+F 0 "#PWR029" H 5050 4450 30  0001 C CNN
 F 1 "GND" H 5050 4380 30  0001 C CNN
 F 2 "" H 5050 4450 60  0000 C CNN
@@
 $EndComp
 $Comp
-L VCC #PWR?
+L VCC #PWR030
 U 1 1 547BBACC
 P 5600 3450
-F 0 "#PWR?" H 5600 3550 30  0001 C CNN
+F 0 "#PWR030" H 5600 3550 30  0001 C CNN
 F 1 "VCC" H 5600 3550 30  0000 C CNN
 F 2 "" H 5600 3450 60  0000 C CNN
@@
 $EndComp
 $Comp
-L VCC #PWR?
+L VCC #PWR031
 U 1 1 547BBAE5
 P 5800 4150
-F 0 "#PWR?" H 5800 4250 30  0001 C CNN
+F 0 "#PWR031" H 5800 4250 30  0001 C CNN
 F 1 "VCC" H 5800 4250 30  0000 C CNN
 F 2 "" H 5800 4150 60  0000 C CNN
