File: project/batfind/filt_out_us.sch (KiCad schematic (older format))
At the start: 0 parts

Commit message: Schematic updated
Parts:
- added C?: 1n, symbol C
- added C?: 1.4u, symbol C
- added R?: 1k, symbol R
- added R?: 10k, symbol R
- added U?: OPA835, symbol OPA835
Connections:
- net filt_in: now also R?.2
- net filt_out: now also C?.1, R?.1
- new net: C?.2, U?.1 (OUT), U?.4 (IN-)
- new net: C?.1, R?.1, U?.3 (IN+)
- new net GND: C?.2, R?.2, U?.2 (VS-)
- new net VCC: U?.5 (PD), U?.6 (VS+)
Changed lines of the file:
@@
 Comment4 ""
 $EndDescr
-Text HLabel 4250 3700 0    60   Input ~ 0
+Text HLabel 4050 3700 0    60   Input ~ 0
 filt_in
-Text HLabel 6650 3650 2    60   Output ~ 0
+Text HLabel 6650 3550 2    60   Output ~ 0
 filt_out
+Text HLabel 4050 4100 0    60   Input ~ 0
+ref
+$Comp
+L OPA835 U?
+U 1 1 547BBD8F
+P 5300 3550
+F 0 "U?" H 5600 3700 60  0000 C CNN
+F 1 "OPA835" H 5700 3400 60  0000 C CNN
+F 2 "" H 5700 3400 60  0000 C CNN
+F 3 "" H 5700 3400 60  0000 C CNN
+	1    5300 3550
+	1    0    0    -1
+$EndComp
+$Comp
+L R R?
+U 1 1 547BBDD1
+P 4450 3700
+F 0 "R?" V 4530 3700 40  0000 C CNN
+F 1 "1k" V 4457 3701 40  0000 C CNN
+F 2 "" V 4380 3700 30  0000 C CNN
+F 3 "" H 4450 3700 30  0000 C CNN
+	1    4450 3700
+	0    1    1    0
+$EndComp
+$Comp
+L R R?
+U 1 1 547BBE10
+P 6550 3850
+F 0 "R?" V 6630 3850 40  0000 C CNN
+F 1 "10k" V 6557 3851 40  0000 C CNN
+F 2 "" V 6480 3850 30  0000 C CNN
+F 3 "" H 6550 3850 30  0000 C CNN
+	1    6550 3850
+	1    0    0    -1
+$EndComp
+$Comp
+L C C?
+U 1 1 547BBE58
+P 4750 3950
+F 0 "C?" H 4750 4050 40  0000 L CNN
+F 1 "1n" H 4756 3865 40  0000 L CNN
+F 2 "" H 4788 3800 30  0000 C CNN
+F 3 "" H 4750 3950 60  0000 C CNN
+	1    4750 3950
+	1    0    0    -1
+$EndComp
+$Comp
+L C C?
+U 1 1 547BBEA7
+P 6200 3550
+F 0 "C?" H 6200 3650 40  0000 L CNN
+F 1 "1.4u" H 6206 3465 40  0000 L CNN
+F 2 "" H 6238 3400 30  0000 C CNN
+F 3 "" H 6200 3550 60  0000 C CNN
+	1    6200 3550
+	0    1    1    0
+$EndComp
+Wire Wire Line
+	4050 3700 4200 3700
+Wire Wire Line
+	4700 3700 4800 3700
+Wire Wire Line
+	4750 3700 4750 3750
+Connection ~ 4750 3700
+Wire Wire Line
+	4800 3400 4650 3400
+Wire Wire Line
+	4650 3400 4650 2850
+Wire Wire Line
+	4650 2850 5950 2850
+Wire Wire Line
+	5950 2850 5950 3550
+Wire Wire Line
+	5900 3550 6000 3550
+Connection ~ 5950 3550
+Wire Wire Line
+	6400 3550 6650 3550
+Wire Wire Line
+	6550 3550 6550 3600
+Connection ~ 6550 3550
+$Comp
+L GND #PWR?
+U 1 1 547BBF4E
+P 6550 4100
+F 0 "#PWR?" H 6550 4100 30  0001 C CNN
+F 1 "GND" H 6550 4030 30  0001 C CNN
+F 2 "" H 6550 4100 60  0000 C CNN
+F 3 "" H 6550 4100 60  0000 C CNN
+	1    6550 4100
+	1    0    0    -1
+$EndComp
+$Comp
+L GND #PWR?
+U 1 1 547BBF67
+P 5250 3950
+F 0 "#PWR?" H 5250 3950 30  0001 C CNN
+F 1 "GND" H 5250 3880 30  0001 C CNN
+F 2 "" H 5250 3950 60  0000 C CNN
+F 3 "" H 5250 3950 60  0000 C CNN
+	1    5250 3950
+	1    0    0    -1
+$EndComp
+$Comp
+L GND #PWR?
+U 1 1 547BBF80
+P 4750 4150
+F 0 "#PWR?" H 4750 4150 30  0001 C CNN
+F 1 "GND" H 4750 4080 30  0001 C CNN
+F 2 "" H 4750 4150 60  0000 C CNN
+F 3 "" H 4750 4150 60  0000 C CNN
+	1    4750 4150
+	1    0    0    -1
+$EndComp
+$Comp
+L VCC #PWR?
+U 1 1 547BBF99
+P 5250 3150
+F 0 "#PWR?" H 5250 3250 30  0001 C CNN
+F 1 "VCC" H 5250 3250 30  0000 C CNN
+F 2 "" H 5250 3150 60  0000 C CNN
+F 3 "" H 5250 3150 60  0000 C CNN
+	1    5250 3150
+	1    0    0    -1
+$EndComp
+$Comp
+L VCC #PWR?
+U 1 1 547BBFB2
+P 5450 3850
+F 0 "#PWR?" H 5450 3950 30  0001 C CNN
+F 1 "VCC" H 5450 3950 30  0000 C CNN
+F 2 "" H 5450 3850 60  0000 C CNN
+F 3 "" H 5450 3850 60  0000 C CNN
+	1    5450 3850
+	-1   0    0    1
+$EndComp
 $EndSCHEMATC

Commit message: Schematic annotated and netlist generated
Parts:
- gave numbers to parts that had none: 5
Changed lines of the file:
@@
 ref
 $Comp
-L OPA835 U?
+L OPA835 U7
 U 1 1 547BBD8F
 P 5300 3550
-F 0 "U?" H 5600 3700 60  0000 C CNN
+F 0 "U7" H 5600 3700 60  0000 C CNN
 F 1 "OPA835" H 5700 3400 60  0000 C CNN
 F 2 "" H 5700 3400 60  0000 C CNN
@@
 $EndComp
 $Comp
-L R R?
+L R R15
 U 1 1 547BBDD1
 P 4450 3700
-F 0 "R?" V 4530 3700 40  0000 C CNN
+F 0 "R15" V 4530 3700 40  0000 C CNN
 F 1 "1k" V 4457 3701 40  0000 C CNN
 F 2 "" V 4380 3700 30  0000 C CNN
@@
 $EndComp
 $Comp
-L R R?
+L R R16
 U 1 1 547BBE10
 P 6550 3850
-F 0 "R?" V 6630 3850 40  0000 C CNN
+F 0 "R16" V 6630 3850 40  0000 C CNN
 F 1 "10k" V 6557 3851 40  0000 C CNN
 F 2 "" V 6480 3850 30  0000 C CNN
@@
 $EndComp
 $Comp
-L C C?
+L C C13
 U 1 1 547BBE58
 P 4750 3950
-F 0 "C?" H 4750 4050 40  0000 L CNN
+F 0 "C13" H 4750 4050 40  0000 L CNN
 F 1 "1n" H 4756 3865 40  0000 L CNN
 F 2 "" H 4788 3800 30  0000 C CNN
@@
 $EndComp
 $Comp
-L C C?
+L C C14
 U 1 1 547BBEA7
 P 6200 3550
-F 0 "C?" H 6200 3650 40  0000 L CNN
+F 0 "C14" H 6200 3650 40  0000 L CNN
 F 1 "1.4u" H 6206 3465 40  0000 L CNN
 F 2 "" H 6238 3400 30  0000 C CNN
@@
 Connection ~ 6550 3550
 $Comp
-L GND #PWR?
+L GND #PWR032
 U 1 1 547BBF4E
 P 6550 4100
-F 0 "#PWR?" H 6550 4100 30  0001 C CNN
+F 0 "#PWR032" H 6550 4100 30  0001 C CNN
 F 1 "GND" H 6550 4030 30  0001 C CNN
 F 2 "" H 6550 4100 60  0000 C CNN
@@
 $EndComp
 $Comp
-L GND #PWR?
+L GND #PWR033
 U 1 1 547BBF67
 P 5250 3950
-F 0 "#PWR?" H 5250 3950 30  0001 C CNN
+F 0 "#PWR033" H 5250 3950 30  0001 C CNN
 F 1 "GND" H 5250 3880 30  0001 C CNN
 F 2 "" H 5250 3950 60  0000 C CNN
@@
 $EndComp
 $Comp
-L GND #PWR?
+L GND #PWR034
 U 1 1 547BBF80
 P 4750 4150
-F 0 "#PWR?" H 4750 4150 30  0001 C CNN
+F 0 "#PWR034" H 4750 4150 30  0001 C CNN
 F 1 "GND" H 4750 4080 30  0001 C CNN
 F 2 "" H 4750 4150 60  0000 C CNN
@@
 $EndComp
 $Comp
-L VCC #PWR?
+L VCC #PWR035
 U 1 1 547BBF99
 P 5250 3150
-F 0 "#PWR?" H 5250 3250 30  0001 C CNN
+F 0 "#PWR035" H 5250 3250 30  0001 C CNN
 F 1 "VCC" H 5250 3250 30  0000 C CNN
 F 2 "" H 5250 3150 60  0000 C CNN
@@
 $EndComp
 $Comp
-L VCC #PWR?
+L VCC #PWR036
 U 1 1 547BBFB2
 P 5450 3850
-F 0 "#PWR?" H 5450 3950 30  0001 C CNN
+F 0 "#PWR036" H 5450 3950 30  0001 C CNN
 F 1 "VCC" H 5450 3950 30  0000 C CNN
 F 2 "" H 5450 3850 60  0000 C CNN
