File: project/batfind/lsp_audio.sch (KiCad schematic (older format))
At the start: 0 parts

Commit message: Schematic updated
Parts:
- added P?: CONN_01X02, symbol CONN_01X02
Connections:
- net lsp_in: now also P?.1 (P1)
- new net GND: P?.2 (P2)
Changed lines of the file:
@@
 Text HLabel 4250 3950 0    60   Input ~ 0
 lsp_in
+$Comp
+L CONN_01X02 P?
+U 1 1 5478EEE7
+P 4950 4000
+F 0 "P?" H 4950 4150 50  0000 C CNN
+F 1 "CONN_01X02" V 5050 4000 50  0000 C CNN
+F 2 "" H 4950 4000 60  0000 C CNN
+F 3 "" H 4950 4000 60  0000 C CNN
+	1    4950 4000
+	1    0    0    -1
+$EndComp
+$Comp
+L GND #PWR?
+U 1 1 5478EF27
+P 4500 4250
+F 0 "#PWR?" H 4500 4250 30  0001 C CNN
+F 1 "GND" H 4500 4180 30  0001 C CNN
+F 2 "" H 4500 4250 60  0000 C CNN
+F 3 "" H 4500 4250 60  0000 C CNN
+	1    4500 4250
+	1    0    0    -1
+$EndComp
+Wire Wire Line
+	4250 3950 4750 3950
+Wire Wire Line
+	4750 4050 4500 4050
+Wire Wire Line
+	4500 4050 4500 4250
 $EndSCHEMATC

Commit message: Schematic annotated and netlist generated
Parts:
- gave numbers to parts that had none: 1
Changed lines of the file:
@@
 lsp_in
 $Comp
-L CONN_01X02 P?
+L CONN_01X02 P5
 U 1 1 5478EEE7
 P 4950 4000
-F 0 "P?" H 4950 4150 50  0000 C CNN
+F 0 "P5" H 4950 4150 50  0000 C CNN
 F 1 "CONN_01X02" V 5050 4000 50  0000 C CNN
 F 2 "" H 4950 4000 60  0000 C CNN
@@
 $EndComp
 $Comp
-L GND #PWR?
+L GND #PWR050
 U 1 1 5478EF27
 P 4500 4250
-F 0 "#PWR?" H 4500 4250 30  0001 C CNN
+F 0 "#PWR050" H 4500 4250 30  0001 C CNN
 F 1 "GND" H 4500 4180 30  0001 C CNN
 F 2 "" H 4500 4250 60  0000 C CNN
