File: project/batfind/lsp_us.sch (KiCad schematic (older format))
At the start: 0 parts

Commit message: Schematic updated
Parts:
- added P?: CONN_01X02, symbol CONN_01X02
Connections:
- net lsp_in: now also P?.1 (P1)
- new net GND: P?.2 (P2)
Changed lines of the file:
@@
 Text HLabel 3750 4000 0    60   Input ~ 0
 lsp_in
+$Comp
+L CONN_01X02 P?
+U 1 1 5478EDD2
+P 4400 4050
+F 0 "P?" H 4400 4200 50  0000 C CNN
+F 1 "CONN_01X02" V 4500 4050 50  0000 C CNN
+F 2 "" H 4400 4050 60  0000 C CNN
+F 3 "" H 4400 4050 60  0000 C CNN
+	1    4400 4050
+	1    0    0    -1
+$EndComp
+$Comp
+L GND #PWR?
+U 1 1 5478EE02
+P 4000 4250
+F 0 "#PWR?" H 4000 4250 30  0001 C CNN
+F 1 "GND" H 4000 4180 30  0001 C CNN
+F 2 "" H 4000 4250 60  0000 C CNN
+F 3 "" H 4000 4250 60  0000 C CNN
+	1    4000 4250
+	1    0    0    -1
+$EndComp
+Wire Wire Line
+	3750 4000 4200 4000
+Wire Wire Line
+	4200 4100 4000 4100
+Wire Wire Line
+	4000 4100 4000 4250
 $EndSCHEMATC

Commit message: Schematic annotated and netlist generated
Parts:
- gave numbers to parts that had none: 1
Changed lines of the file:
@@
 lsp_in
 $Comp
-L CONN_01X02 P?
+L CONN_01X02 P4
 U 1 1 5478EDD2
 P 4400 4050
-F 0 "P?" H 4400 4200 50  0000 C CNN
+F 0 "P4" H 4400 4200 50  0000 C CNN
 F 1 "CONN_01X02" V 4500 4050 50  0000 C CNN
 F 2 "" H 4400 4050 60  0000 C CNN
@@
 $EndComp
 $Comp
-L GND #PWR?
+L GND #PWR049
 U 1 1 5478EE02
 P 4000 4250
-F 0 "#PWR?" H 4000 4250 30  0001 C CNN
+F 0 "#PWR049" H 4000 4250 30  0001 C CNN
 F 1 "GND" H 4000 4180 30  0001 C CNN
 F 2 "" H 4000 4250 60  0000 C CNN
