File: project/batfind/mic_audio.sch (KiCad schematic (older format))
At the start: 0 parts

Commit message: Schematic updated
Parts:
- added C?: C, symbol C
- added P?: CONN_01X02, symbol CONN_01X02
- added R?: R, symbol R
Connections:
- net mic_out: now also C?.1, R?.1
- new net: C?.2, P?.1 (P1)
- new net GND: P?.2 (P2)
- new net ref: R?.2
Changed lines of the file:
@@
 Text HLabel 6600 4200 2    60   Output ~ 0
 mic_out
+$Comp
+L CONN_01X02 P?
+U 1 1 5478C6A6
+P 5350 4250
+F 0 "P?" H 5350 4400 50  0000 C CNN
+F 1 "CONN_01X02" V 5450 4250 50  0000 C CNN
+F 2 "" H 5350 4250 60  0000 C CNN
+F 3 "" H 5350 4250 60  0000 C CNN
+	1    5350 4250
+	-1   0    0    -1
+$EndComp
+$Comp
+L GND #PWR?
+U 1 1 5478C6E0
+P 5750 4450
+F 0 "#PWR?" H 5750 4450 30  0001 C CNN
+F 1 "GND" H 5750 4380 30  0001 C CNN
+F 2 "" H 5750 4450 60  0000 C CNN
+F 3 "" H 5750 4450 60  0000 C CNN
+	1    5750 4450
+	1    0    0    -1
+$EndComp
+Wire Wire Line
+	5750 4450 5750 4300
+Wire Wire Line
+	5750 4300 5550 4300
+$Comp
+L C C?
+U 1 1 5478C6F8
+P 5950 4200
+F 0 "C?" H 5950 4300 40  0000 L CNN
+F 1 "C" H 5956 4115 40  0000 L CNN
+F 2 "" H 5988 4050 30  0000 C CNN
+F 3 "" H 5950 4200 60  0000 C CNN
+	1    5950 4200
+	0    1    1    0
+$EndComp
+Wire Wire Line
+	5750 4200 5550 4200
+Wire Wire Line
+	6150 4200 6600 4200
+Text HLabel 6350 4950 3    60   Input ~ 0
+ref
+$Comp
+L R R?
+U 1 1 5478C821
+P 6350 4550
+F 0 "R?" V 6430 4550 40  0000 C CNN
+F 1 "R" V 6357 4551 40  0000 C CNN
+F 2 "" V 6280 4550 30  0000 C CNN
+F 3 "" H 6350 4550 30  0000 C CNN
+	1    6350 4550
+	1    0    0    -1
+$EndComp
+Wire Wire Line
+	6350 4300 6350 4200
+Connection ~ 6350 4200
+Wire Wire Line
+	6350 4950 6350 4800
 $EndSCHEMATC

Commit message: Schematic annotated and netlist generated
Parts:
- gave numbers to parts that had none: 3
Changed lines of the file:
@@
 mic_out
 $Comp
-L CONN_01X02 P?
+L CONN_01X02 P3
 U 1 1 5478C6A6
 P 5350 4250
-F 0 "P?" H 5350 4400 50  0000 C CNN
+F 0 "P3" H 5350 4400 50  0000 C CNN
 F 1 "CONN_01X02" V 5450 4250 50  0000 C CNN
 F 2 "" H 5350 4250 60  0000 C CNN
@@
 $EndComp
 $Comp
-L GND #PWR?
+L GND #PWR048
 U 1 1 5478C6E0
 P 5750 4450
-F 0 "#PWR?" H 5750 4450 30  0001 C CNN
+F 0 "#PWR048" H 5750 4450 30  0001 C CNN
 F 1 "GND" H 5750 4380 30  0001 C CNN
 F 2 "" H 5750 4450 60  0000 C CNN
@@
 	5750 4300 5550 4300
 $Comp
-L C C?
+L C C20
 U 1 1 5478C6F8
 P 5950 4200
-F 0 "C?" H 5950 4300 40  0000 L CNN
+F 0 "C20" H 5950 4300 40  0000 L CNN
 F 1 "C" H 5956 4115 40  0000 L CNN
 F 2 "" H 5988 4050 30  0000 C CNN
@@
 ref
 $Comp
-L R R?
+L R R22
 U 1 1 5478C821
 P 6350 4550
-F 0 "R?" V 6430 4550 40  0000 C CNN
+F 0 "R22" V 6430 4550 40  0000 C CNN
 F 1 "R" V 6357 4551 40  0000 C CNN
 F 2 "" V 6280 4550 30  0000 C CNN
