File: project/batfind/mult.sch (KiCad schematic (older format))
At the start: 15 parts

Commit message: Schematic updated
Parts:
- added C?: 27n, symbol C
- added C?: 10n, symbol C
- added R? (x2): 68, symbol R
- added R?: 30, symbol R
- added U?: OPA835, symbol OPA835
- R? (x2): value R -> 10k
Connections:
- wire segments 33 -> 44
Changed lines of the file:
@@
 	1    0    0    -1
 $EndComp
-Text HLabel 8050 2400 2    60   Output ~ 0
+Text HLabel 10350 2550 2    60   Output ~ 0
 AxB
 $Comp
@@
 Connection ~ 6700 4700
 Wire Wire Line
-	2300 5400 6700 5400
+	2300 5400 8850 5400
 Wire Wire Line
 	6700 5400 6700 5300
@@
 P 4050 1800
 F 0 "R?" V 4130 1800 40  0000 C CNN
-F 1 "R" V 4057 1801 40  0000 C CNN
+F 1 "10k" V 4057 1801 40  0000 C CNN
 F 2 "" V 3980 1800 30  0000 C CNN
 F 3 "" H 4050 1800 30  0000 C CNN
@@
 P 4900 1300
 F 0 "R?" V 4980 1300 40  0000 C CNN
-F 1 "R" V 4907 1301 40  0000 C CNN
+F 1 "10k" V 4907 1301 40  0000 C CNN
 F 2 "" V 4830 1300 30  0000 C CNN
 F 3 "" H 4900 1300 30  0000 C CNN
@@
 	5550 1950 5700 1950
 Connection ~ 5700 1950
-Wire Wire Line
-	7700 2400 8050 2400
 $Comp
 L C C?
@@
 	1    0    0    -1
 $EndComp
+$Comp
+L R R?
+U 1 1 54786A98
+P 8050 2400
+F 0 "R?" V 8130 2400 40  0000 C CNN
+F 1 "68" V 8057 2401 40  0000 C CNN
+F 2 "" V 7980 2400 30  0000 C CNN
+F 3 "" H 8050 2400 30  0000 C CNN
+	1    8050 2400
+	0    1    1    0
+$EndComp
+$Comp
+L OPA835 U?
+U 1 1 54786F37
+P 9500 2550
+F 0 "U?" H 9800 2700 60  0000 C CNN
+F 1 "OPA835" H 9900 2400 60  0000 C CNN
+F 2 "" H 9900 2400 60  0000 C CNN
+F 3 "" H 9900 2400 60  0000 C CNN
+	1    9500 2550
+	1    0    0    -1
+$EndComp
+$Comp
+L R R?
+U 1 1 547871B1
+P 8650 2400
+F 0 "R?" V 8730 2400 40  0000 C CNN
+F 1 "30" V 8657 2401 40  0000 C CNN
+F 2 "" V 8580 2400 30  0000 C CNN
+F 3 "" H 8650 2400 30  0000 C CNN
+	1    8650 2400
+	0    1    1    0
+$EndComp
+$Comp
+L R R?
+U 1 1 547871EB
+P 8350 2100
+F 0 "R?" V 8430 2100 40  0000 C CNN
+F 1 "68" V 8357 2101 40  0000 C CNN
+F 2 "" V 8280 2100 30  0000 C CNN
+F 3 "" H 8350 2100 30  0000 C CNN
+	1    8350 2100
+	-1   0    0    1
+$EndComp
+$Comp
+L C C?
+U 1 1 54787233
+P 8350 2650
+F 0 "C?" H 8350 2750 40  0000 L CNN
+F 1 "27n" H 8356 2565 40  0000 L CNN
+F 2 "" H 8388 2500 30  0000 C CNN
+F 3 "" H 8350 2650 60  0000 C CNN
+	1    8350 2650
+	1    0    0    -1
+$EndComp
+$Comp
+L C C?
+U 1 1 54787284
+P 8950 2150
+F 0 "C?" H 8950 2250 40  0000 L CNN
+F 1 "10n" H 8956 2065 40  0000 L CNN
+F 2 "" H 8988 2000 30  0000 C CNN
+F 3 "" H 8950 2150 60  0000 C CNN
+	1    8950 2150
+	1    0    0    -1
+$EndComp
+Wire Wire Line
+	7700 2400 7800 2400
+Wire Wire Line
+	8300 2400 8400 2400
+Wire Wire Line
+	8350 2350 8350 2450
+Connection ~ 8350 2400
+Wire Wire Line
+	8350 1850 8350 1750
+Wire Wire Line
+	8350 1750 10200 1750
+Wire Wire Line
+	10200 1750 10200 2550
+Wire Wire Line
+	10100 2550 10350 2550
+Connection ~ 10200 2550
+Wire Wire Line
+	8950 1950 8950 1750
+Connection ~ 8950 1750
+Wire Wire Line
+	8900 2400 9000 2400
+Wire Wire Line
+	8950 2350 8950 2400
+Connection ~ 8950 2400
+Wire Wire Line
+	8850 5400 8850 2700
+Wire Wire Line
+	8850 2700 9000 2700
+Connection ~ 6700 5400
+$Comp
+L VCC #PWR?
+U 1 1 547878DE
+P 9450 2150
+F 0 "#PWR?" H 9450 2250 30  0001 C CNN
+F 1 "VCC" H 9450 2250 30  0000 C CNN
+F 2 "" H 9450 2150 60  0000 C CNN
+F 3 "" H 9450 2150 60  0000 C CNN
+	1    9450 2150
+	1    0    0    -1
+$EndComp
+$Comp
+L GND #PWR?
+U 1 1 54787C5B
+P 9450 2950
+F 0 "#PWR?" H 9450 2950 30  0001 C CNN
+F 1 "GND" H 9450 2880 30  0000 C CNN
+F 2 "" H 9450 2950 60  0000 C CNN
+F 3 "" H 9450 2950 60  0000 C CNN
+	1    9450 2950
+	1    0    0    -1
+$EndComp
+$Comp
+L VCC #PWR?
+U 1 1 54787F06
+P 9650 2850
+F 0 "#PWR?" H 9650 2950 30  0001 C CNN
+F 1 "VCC" H 9650 2950 30  0000 C CNN
+F 2 "" H 9650 2850 60  0000 C CNN
+F 3 "" H 9650 2850 60  0000 C CNN
+	1    9650 2850
+	-1   0    0    1
+$EndComp
+$Comp
+L GND #PWR?
+U 1 1 5478B491
+P 8350 2850
+F 0 "#PWR?" H 8350 2850 30  0001 C CNN
+F 1 "GND" H 8350 2780 30  0000 C CNN
+F 2 "" H 8350 2850 60  0000 C CNN
+F 3 "" H 8350 2850 60  0000 C CNN
+	1    8350 2850
+	1    0    0    -1
+$EndComp

Commit message: Schematic annotated and netlist generated
Parts:
- gave numbers to parts that had none: 21
