File: project/batfind/sine.sch (KiCad schematic (older format))
At the start: 0 parts

Commit message: Schematic updated
Parts:
- added C?: C, symbol C
- added P?: CONN_01X02, symbol CONN_01X02
- added R?: R, symbol R
Connections:
- net ref: now also R?.2
- net sine: now also C?.1, R?.1
- new net: C?.2, P?.1 (P1)
- new net GND: P?.2 (P2)
Changed lines of the file:
@@
 Comment4 ""
 $EndDescr
-Text HLabel 3050 4550 0    60   Input ~ 0
+Text HLabel 5600 4700 3    60   Input ~ 0
 ref
-Text HLabel 5250 4000 2    60   Output ~ 0
+Text HLabel 5800 4000 2    60   Output ~ 0
 sine
+$Comp
+L CONN_01X02 P?
+U 1 1 5478B984
+P 4800 4050
+F 0 "P?" H 4800 4200 50  0000 C CNN
+F 1 "CONN_01X02" V 4900 4050 50  0000 C CNN
+F 2 "" H 4800 4050 60  0000 C CNN
+F 3 "" H 4800 4050 60  0000 C CNN
+	1    4800 4050
+	-1   0    0    -1
+$EndComp
+$Comp
+L GND #PWR?
+U 1 1 5478B9D5
+P 5150 4250
+F 0 "#PWR?" H 5150 4250 30  0001 C CNN
+F 1 "GND" H 5150 4180 30  0001 C CNN
+F 2 "" H 5150 4250 60  0000 C CNN
+F 3 "" H 5150 4250 60  0000 C CNN
+	1    5150 4250
+	1    0    0    -1
+$EndComp
+$Comp
+L R R?
+U 1 1 5478F0D7
+P 5600 4300
+F 0 "R?" V 5680 4300 40  0000 C CNN
+F 1 "R" V 5607 4301 40  0000 C CNN
+F 2 "" V 5530 4300 30  0000 C CNN
+F 3 "" H 5600 4300 30  0000 C CNN
+	1    5600 4300
+	1    0    0    -1
+$EndComp
+$Comp
+L C C?
+U 1 1 5478F106
+P 5300 4000
+F 0 "C?" H 5300 4100 40  0000 L CNN
+F 1 "C" H 5306 3915 40  0000 L CNN
+F 2 "" H 5338 3850 30  0000 C CNN
+F 3 "" H 5300 4000 60  0000 C CNN
+	1    5300 4000
+	0    1    1    0
+$EndComp
+Wire Wire Line
+	5000 4000 5100 4000
+Wire Wire Line
+	5500 4000 5800 4000
+Wire Wire Line
+	5600 4000 5600 4050
+Connection ~ 5600 4000
+Wire Wire Line
+	5600 4550 5600 4700
+Wire Wire Line
+	5000 4100 5150 4100
+Wire Wire Line
+	5150 4100 5150 4250
 $EndSCHEMATC

Commit message: Schematic annotated and netlist generated
Parts:
- gave numbers to parts that had none: 3
Changed lines of the file:
@@
 sine
 $Comp
-L CONN_01X02 P?
+L CONN_01X02 P1
 U 1 1 5478B984
 P 4800 4050
-F 0 "P?" H 4800 4200 50  0000 C CNN
+F 0 "P1" H 4800 4200 50  0000 C CNN
 F 1 "CONN_01X02" V 4900 4050 50  0000 C CNN
 F 2 "" H 4800 4050 60  0000 C CNN
@@
 $EndComp
 $Comp
-L GND #PWR?
+L GND #PWR022
 U 1 1 5478B9D5
 P 5150 4250
-F 0 "#PWR?" H 5150 4250 30  0001 C CNN
+F 0 "#PWR022" H 5150 4250 30  0001 C CNN
 F 1 "GND" H 5150 4180 30  0001 C CNN
 F 2 "" H 5150 4250 60  0000 C CNN
@@
 $EndComp
 $Comp
-L R R?
+L R R10
 U 1 1 5478F0D7
 P 5600 4300
-F 0 "R?" V 5680 4300 40  0000 C CNN
+F 0 "R10" V 5680 4300 40  0000 C CNN
 F 1 "R" V 5607 4301 40  0000 C CNN
 F 2 "" V 5530 4300 30  0000 C CNN
@@
 $EndComp
 $Comp
-L C C?
+L C C8
 U 1 1 5478F106
 P 5300 4000
-F 0 "C?" H 5300 4100 40  0000 L CNN
+F 0 "C8" H 5300 4100 40  0000 L CNN
 F 1 "C" H 5306 3915 40  0000 L CNN
 F 2 "" H 5338 3850 30  0000 C CNN
