File: project/batfind/sw_in.sch (KiCad schematic (older format))
At the start: 0 parts

Commit message: Schematic updated
Parts:
- added GS?: GS3, GS3, symbol GS3
Connections:
- net sw_a: now also GS?.1 (G1)
- net sw_b: now also GS?.3 (G3)
- net sw_out: now also GS?.2 (G2)
Changed lines of the file:
@@
 Comment4 ""
 $EndDescr
-Text HLabel 5500 3850 2    60   Output ~ 0
+Text HLabel 4400 3900 2    60   Output ~ 0
 sw_out
 Text HLabel 3700 3800 0    60   Input ~ 0
 sw_a
-Text HLabel 3700 4050 0    60   Input ~ 0
+Text HLabel 3700 4000 0    60   Input ~ 0
 sw_b
+Text HLabel 3700 4300 0    60   Input ~ 0
+ref
+$Comp
+L GS3 GS?
+U 1 1 5478B6F4
+P 4050 3900
+F 0 "GS?" H 4100 4100 50  0000 C CNN
+F 1 "GS3" H 4100 3701 40  0000 C CNN
+F 2 "GS3" V 4138 3826 30  0000 C CNN
+F 3 "" H 4050 3900 60  0000 C CNN
+	1    4050 3900
+	1    0    0    -1
+$EndComp
+Wire Wire Line
+	3700 3800 3900 3800
+Wire Wire Line
+	3700 4000 3900 4000
+Wire Wire Line
+	4200 3900 4400 3900
 $EndSCHEMATC

Commit message: Schematic annotated and netlist generated
Parts:
- gave numbers to parts that had none: 1
Changed lines of the file:
@@
 ref
 $Comp
-L GS3 GS?
+L GS3 GS1
 U 1 1 5478B6F4
 P 4050 3900
-F 0 "GS?" H 4100 4100 50  0000 C CNN
+F 0 "GS1" H 4100 4100 50  0000 C CNN
 F 1 "GS3" H 4100 3701 40  0000 C CNN
 F 2 "GS3" V 4138 3826 30  0000 C CNN
