File: project/batfind/sw_out.sch (KiCad schematic (older format))
At the start: 0 parts

Commit message: Schematic updated
Parts:
- added GS?: GS3, GS3, symbol GS3
Connections:
- net sw_in: now also GS?.2 (G2)
- net sw_out_a: now also GS?.1 (G1)
- net sw_out_b: now also GS?.3 (G3)
Changed lines of the file:
@@
 Text HLabel 4200 3750 0    60   Input ~ 0
 sw_in
-Text HLabel 6650 3800 2    60   Output ~ 0
+Text HLabel 4950 3650 2    60   Output ~ 0
 sw_out_a
-Text HLabel 6700 4200 2    60   Output ~ 0
+Text HLabel 4950 3850 2    60   Output ~ 0
 sw_out_b
+Text HLabel 4200 4100 0    60   Input ~ 0
+ref
+$Comp
+L GS3 GS?
+U 1 1 5478B803
+P 4600 3750
+F 0 "GS?" H 4650 3950 50  0000 C CNN
+F 1 "GS3" H 4650 3551 40  0000 C CNN
+F 2 "GS3" V 4688 3676 30  0000 C CNN
+F 3 "" H 4600 3750 60  0000 C CNN
+	1    4600 3750
+	-1   0    0    -1
+$EndComp
+Wire Wire Line
+	4200 3750 4450 3750
+Wire Wire Line
+	4750 3650 4950 3650
+Wire Wire Line
+	4750 3850 4950 3850
 $EndSCHEMATC

Commit message: Schematic annotated and netlist generated
Parts:
- gave numbers to parts that had none: 1
Changed lines of the file:
@@
 ref
 $Comp
-L GS3 GS?
+L GS3 GS2
 U 1 1 5478B803
 P 4600 3750
-F 0 "GS?" H 4650 3950 50  0000 C CNN
+F 0 "GS2" H 4650 3950 50  0000 C CNN
 F 1 "GS3" H 4650 3551 40  0000 C CNN
 F 2 "GS3" V 4688 3676 30  0000 C CNN
